Commit message: remove not used file

File: urdf/ur5_arm/ur5.gazebo.xacro (robot description, xacro)
@@ -1,3 +1,6 @@
 <?xml version="1.0"?>
 <robot xmlns:xacro="http://www.ros.org/wiki/xacro">
+  <xacro:macro name="ur5_arm_gazebo" params="prefix">
+    <!-- nothing to do here at the moment -->
+  </xacro:macro>
 </robot>
